File: KiCad/Tank_Sys/Pump_Sys.sch (KiCad schematic (older format))
At the start: 11 parts, among them K1 AZ7709T-1AE-12DE, M1 12V Pump, Q1 BS170, SW1 SW_SPDT

Commit message: Home update
Parts:
- added J3: Conn_01x04, symbol Connector_Generic:Conn_01x04
- C1: footprint Capacitor_THT:CP_Radial_D4.0mm_P2.00mm -> (none)
- D1, D4: footprint LED_THT:LED_D1.8mm_W1.8mm_H2.4mm_Horizontal_O1.27mm_Z1.6mm -> (none)
- D2, D3: footprint Diode_THT:D_5KPW_P12.70mm_Horizontal -> (none)
- M1: footprint Connector_PinHeader_2.54mm:PinHeader_1x04_P2.54mm_Vertical -> (none)
- R1, R2: footprint Resistor_THT:R_Axial_DIN0204_L3.6mm_D1.6mm_P5.08mm_Horizontal -> (none)
Connections:
- net +12V: now also J3.1 (Pin_1)
- net GND: now also J3.4 (Pin_4)
- net PUMP_CTRL: no longer names the net of Q1.2 (G), R2.1
- net PUMP_CTRL: now also J3.3 (Pin_3)
- net PUMP_SENSE: no longer names the net of D3.2 (A)
- net PUMP_SENSE: now also J3.2 (Pin_2)
Changed lines of the file:
@@
 $Descr A4 11693 8268
 encoding utf-8
-Sheet 1 1
+Sheet 2 3
 Title ""
 Date ""
@@
 F 0 "M1" H 5458 2896 50  0000 L CNN
 F 1 "12V Pump" H 5458 2805 50  0000 L CNN
-F 2 "Connector_PinHeader_2.54mm:PinHeader_1x04_P2.54mm_Vertical" H 5300 2810 50  0001 C CNN
+F 2 "" H 5300 2810 50  0001 C CNN
 F 3 "~" H 5300 2810 50  0001 C CNN
 	1    5300 2900
@@
 F 0 "D2" V 4904 3030 50  0000 L CNN
 F 1 "D" V 4995 3030 50  0000 L CNN
-F 2 "Diode_THT:D_5KPW_P12.70mm_Horizontal" H 4950 2950 50  0001 C CNN
+F 2 "" H 4950 2950 50  0001 C CNN
 F 3 "~" H 4950 2950 50  0001 C CNN
 	1    4950 2950
@@
 	4950 2700 5300 2700
 $Comp
-L power:+12V #PWR0101
+L power:+12V #PWR0109
 U 1 1 61011034
 P 5800 3850
-F 0 "#PWR0101" H 5800 3700 50  0001 C CNN
+F 0 "#PWR0109" H 5800 3700 50  0001 C CNN
 F 1 "+12V" H 5815 4023 50  0000 C CNN
 F 2 "" H 5800 3850 50  0001 C CNN
@@
 $EndComp
 $Comp
-L power:+12V #PWR0102
+L power:+12V #PWR0110
 U 1 1 6101103A
 P 5300 2600
-F 0 "#PWR0102" H 5300 2450 50  0001 C CNN
+F 0 "#PWR0110" H 5300 2450 50  0001 C CNN
 F 1 "+12V" H 5315 2773 50  0000 C CNN
 F 2 "" H 5300 2600 50  0001 C CNN
@@
 $EndComp
 $Comp
-L power:GND #PWR0103
+L power:GND #PWR0111
 U 1 1 61011040
 P 5800 5100
-F 0 "#PWR0103" H 5800 4850 50  0001 C CNN
+F 0 "#PWR0111" H 5800 4850 50  0001 C CNN
 F 1 "GND" H 5805 4927 50  0000 C CNN
 F 2 "" H 5800 5100 50  0001 C CNN
@@
 F 0 "D3" V 5554 3480 50  0000 L CNN
 F 1 "D" V 5645 3480 50  0000 L CNN
-F 2 "Diode_THT:D_5KPW_P12.70mm_Horizontal" H 5600 3400 50  0001 C CNN
+F 2 "" H 5600 3400 50  0001 C CNN
 F 3 "~" H 5600 3400 50  0001 C CNN
 	1    5600 3400
@@
 	5800 5050 5800 5100
 $Comp
-L power:GND #PWR0104
+L power:GND #PWR0112
 U 1 1 61011066
 P 5400 4650
-F 0 "#PWR0104" H 5400 4400 50  0001 C CNN
+F 0 "#PWR0112" H 5400 4400 50  0001 C CNN
 F 1 "GND" H 5405 4477 50  0000 C CNN
 F 2 "" H 5400 4650 50  0001 C CNN
@@
 $EndComp
 $Comp
-L power:GND #PWR0105
+L power:GND #PWR0113
 U 1 1 6101106C
 P 5000 3950
-F 0 "#PWR0105" H 5000 3700 50  0001 C CNN
+F 0 "#PWR0113" H 5000 3700 50  0001 C CNN
 F 1 "GND" H 5005 3777 50  0000 C CNN
 F 2 "" H 5000 3950 50  0001 C CNN
@@
 	5400 3850 5400 3950
 Wire Wire Line
-	5750 3400 6450 3400
-Wire Wire Line
 	5000 3950 5200 3950
 Wire Wire Line
 	5200 3950 5200 3850
-Text HLabel 6250 4850 2    50   Input ~ 0
-PUMP_CTRL
-Text HLabel 6450 3400 2    50   Output ~ 0
-PUMP_SENSE
 $Comp
 L Device:R R2
@@
 F 0 "R2" H 6220 5096 50  0000 L CNN
 F 1 "R" H 6220 5005 50  0000 L CNN
-F 2 "Resistor_THT:R_Axial_DIN0204_L3.6mm_D1.6mm_P5.08mm_Horizontal" V 6080 5050 50  0001 C CNN
+F 2 "" V 6080 5050 50  0001 C CNN
 F 3 "~" H 6150 5050 50  0001 C CNN
 	1    6150 5050
@@
 F 0 "D4" V 6189 5282 50  0000 R CNN
 F 1 "LED" V 6098 5282 50  0000 R CNN
-F 2 "LED_THT:LED_D1.8mm_W1.8mm_H2.4mm_Horizontal_O1.27mm_Z1.6mm" H 6150 5400 50  0001 C CNN
+F 2 "" H 6150 5400 50  0001 C CNN
 F 3 "~" H 6150 5400 50  0001 C CNN
 	1    6150 5400
@@
 AR Path="/60E699EC/60E67611" Ref="#PWR?"  Part="1"
 AR Path="/60FE860F/60E67611" Ref="#PWR?"  Part="1"
-AR Path="/6100D536/60E67611" Ref="#PWR?"  Part="1"
-AR Path="/60E67611" Ref="#PWR0106"  Part="1"
-F 0 "#PWR0106" H 6150 5350 50  0001 C CNN
+AR Path="/6100D536/60E67611" Ref="#PWR0114"  Part="1"
+F 0 "#PWR0114" H 6150 5350 50  0001 C CNN
 F 1 "GND" H 6155 5427 50  0000 C CNN
 F 2 "" H 6150 5600 50  0001 C CNN
@@
 F 0 "R1" H 4720 2896 50  0000 L CNN
 F 1 "R" H 4720 2805 50  0000 L CNN
-F 2 "Resistor_THT:R_Axial_DIN0204_L3.6mm_D1.6mm_P5.08mm_Horizontal" V 4580 2850 50  0001 C CNN
+F 2 "" V 4580 2850 50  0001 C CNN
 F 3 "~" H 4650 2850 50  0001 C CNN
 	1    4650 2850
@@
 F 0 "D1" V 4689 3082 50  0000 R CNN
 F 1 "LED" V 4598 3082 50  0000 R CNN
-F 2 "LED_THT:LED_D1.8mm_W1.8mm_H2.4mm_Horizontal_O1.27mm_Z1.6mm" H 4650 3200 50  0001 C CNN
+F 2 "" H 4650 3200 50  0001 C CNN
 F 3 "~" H 4650 3200 50  0001 C CNN
 	1    4650 3200
@@
 F 0 "C1" H 4765 3596 50  0000 L CNN
 F 1 "C" H 4765 3505 50  0000 L CNN
-F 2 "Capacitor_THT:CP_Radial_D4.0mm_P2.00mm" H 4688 3400 50  0001 C CNN
+F 2 "" H 4688 3400 50  0001 C CNN
 F 3 "~" H 4650 3550 50  0001 C CNN
 	1    4650 3550
@@
 Connection ~ 4650 3400
 $Comp
-L power:GND #PWR0107
+L power:GND #PWR0115
 U 1 1 60E6B091
 P 4650 3750
-F 0 "#PWR0107" H 4650 3500 50  0001 C CNN
+F 0 "#PWR0115" H 4650 3500 50  0001 C CNN
 F 1 "GND" H 4655 3577 50  0000 C CNN
 F 2 "" H 4650 3750 50  0001 C CNN
@@
 Wire Wire Line
 	4650 3750 4650 3700
+$Comp
+L Connector_Generic:Conn_01x04 J3
+U 1 1 614693D4
+P 7400 3600
+F 0 "J3" H 7480 3592 50  0000 L CNN
+F 1 "Conn_01x04" H 7480 3501 50  0000 L CNN
+F 2 "" H 7400 3600 50  0001 C CNN
+F 3 "~" H 7400 3600 50  0001 C CNN
+	1    7400 3600
+	1    0    0    -1
+$EndComp
+$Comp
+L power:+12V #PWR0119
+U 1 1 6146A3C0
+P 7000 3350
+F 0 "#PWR0119" H 7000 3200 50  0001 C CNN
+F 1 "+12V" H 7015 3523 50  0000 C CNN
+F 2 "" H 7000 3350 50  0001 C CNN
+F 3 "" H 7000 3350 50  0001 C CNN
+	1    7000 3350
+	1    0    0    -1
+$EndComp
+$Comp
+L power:GND #PWR?
+U 1 1 6146AE65
+P 7050 3900
+AR Path="/60E68C49/6146AE65" Ref="#PWR?"  Part="1"
+AR Path="/60E68E60/6146AE65" Ref="#PWR?"  Part="1"
+AR Path="/60E68F4B/6146AE65" Ref="#PWR?"  Part="1"
+AR Path="/60E699AB/6146AE65" Ref="#PWR?"  Part="1"
+AR Path="/60E699EC/6146AE65" Ref="#PWR?"  Part="1"
+AR Path="/60FE860F/6146AE65" Ref="#PWR?"  Part="1"
+AR Path="/6100D536/6146AE65" Ref="#PWR0120"  Part="1"
+F 0 "#PWR0120" H 7050 3650 50  0001 C CNN
+F 1 "GND" H 7055 3727 50  0000 C CNN
+F 2 "" H 7050 3900 50  0001 C CNN
+F 3 "" H 7050 3900 50  0001 C CNN
+	1    7050 3900
+	1    0    0    -1
+$EndComp
+Wire Wire Line
+	7200 3800 7050 3800
+Wire Wire Line
+	7050 3800 7050 3900
+Wire Wire Line
+	7200 3700 6250 3700
+Wire Wire Line
+	6250 3700 6250 4850
+Wire Wire Line
+	7200 3600 6000 3600
+Wire Wire Line
+	6000 3600 6000 3400
+Wire Wire Line
+	6000 3400 5750 3400
+Wire Wire Line
+	7000 3500 7200 3500
+Wire Wire Line
+	7000 3350 7000 3500
 $EndSCHEMATC
