File: KiCad/Tank_Sys/Tank_Sys.sch (KiCad schematic (older format))
At the start: 5 parts

Commit message: Home update
Parts:
- U1: renamed from U?; symbol Arduino:Arduino_Pro_Mini -> Tank_Sys-rescue:Arduino_Pro_Mini-Arduino
- U2: renamed from U?; symbol ESP8266:ESP-01v090 -> Tank_Sys-rescue:ESP-01v090-ESP8266
- U3: renamed from U?; footprint 78XXL -> Common:VREG_TO-220-3; symbol SparkFun-IC-Power:V_REG_LD1117VXX -> Tank_Sys-rescue:V_REG_LD1117VXX-SparkFun-IC-Power
- gave numbers to parts that had none: 2
Changed lines of the file:
@@
 $EndDescr
 $Comp
-L Arduino:Arduino_Pro_Mini U?
+L Tank_Sys-rescue:Arduino_Pro_Mini-Arduino U1
 U 1 1 60E5DA35
 P 3250 3100
-F 0 "U?" H 3250 3989 60  0000 C CNN
+F 0 "U1" H 3250 3989 60  0000 C CNN
 F 1 "Arduino_Pro_Mini" H 3250 3883 60  0000 C CNN
 F 2 "Arduino:Arduino_Pro_Mini" H 4050 2350 60  0001 C CNN
@@
 $EndComp
 $Comp
-L Connector:Barrel_Jack J?
+L Connector:Barrel_Jack J1
 U 1 1 60E63BA5
 P 1400 1300
-F 0 "J?" H 1457 1625 50  0000 C CNN
+F 0 "J1" H 1457 1625 50  0000 C CNN
 F 1 "Barrel_Jack" H 1457 1534 50  0000 C CNN
 F 2 "" H 1450 1260 50  0001 C CNN
@@
 $EndComp
 $Comp
-L power:+12V #PWR?
+L power:+12V #PWR0101
 U 1 1 60E65AA3
 P 1850 1050
-F 0 "#PWR?" H 1850 900 50  0001 C CNN
+F 0 "#PWR0101" H 1850 900 50  0001 C CNN
 F 1 "+12V" H 1865 1223 50  0000 C CNN
 F 2 "" H 1850 1050 50  0001 C CNN
@@
 $EndComp
 $Comp
-L power:GND #PWR?
+L power:GND #PWR0102
 U 1 1 60E66776
 P 1850 1500
-F 0 "#PWR?" H 1850 1250 50  0001 C CNN
+F 0 "#PWR0102" H 1850 1250 50  0001 C CNN
 F 1 "GND" H 1855 1327 50  0000 C CNN
 F 2 "" H 1850 1500 50  0001 C CNN
@@
 	1850 1400 1850 1500
 $Comp
-L power:+12V #PWR?
+L power:+12V #PWR0103
 U 1 1 60E67415
 P 4050 2500
-F 0 "#PWR?" H 4050 2350 50  0001 C CNN
+F 0 "#PWR0103" H 4050 2350 50  0001 C CNN
 F 1 "+12V" H 4065 2673 50  0000 C CNN
 F 2 "" H 4050 2500 50  0001 C CNN
@@
 $EndComp
 $Comp
-L power:GND #PWR?
+L power:GND #PWR0104
 U 1 1 60E67CFD
 P 3950 2600
-F 0 "#PWR?" H 3950 2350 50  0001 C CNN
+F 0 "#PWR0104" H 3950 2350 50  0001 C CNN
 F 1 "GND" H 3955 2427 50  0000 C CNN
 F 2 "" H 3950 2600 50  0001 C CNN
@@
 $EndComp
 $Comp
-L ESP8266:ESP-01v090 U?
+L Tank_Sys-rescue:ESP-01v090-ESP8266 U2
 U 1 1 60E6BB22
 P 8350 3350
-F 0 "U?" H 8350 3865 50  0000 C CNN
+F 0 "U2" H 8350 3865 50  0000 C CNN
 F 1 "ESP-01v090" H 8350 3774 50  0000 C CNN
 F 2 "" H 8350 3350 50  0001 C CNN
@@
 	10600 1300 10450 1300
 $Comp
-L power:GND #PWR?
+L power:GND #PWR0105
 U 1 1 60E7792E
 P 10150 1800
-F 0 "#PWR?" H 10150 1550 50  0001 C CNN
+F 0 "#PWR0105" H 10150 1550 50  0001 C CNN
 F 1 "GND" H 10155 1627 50  0000 C CNN
 F 2 "" H 10150 1800 50  0001 C CNN
@@
 	9300 2600 9300 3200
 $Comp
-L SparkFun-IC-Power:V_REG_LD1117VXX U?
+L Tank_Sys-rescue:V_REG_LD1117VXX-SparkFun-IC-Power U3
 U 1 1 60E751B1
 P 10150 1300
-F 0 "U?" H 10150 1554 45  0000 C CNN
+F 0 "U3" H 10150 1554 45  0000 C CNN
 F 1 "V_REG_LD1117V33" H 10150 1470 45  0000 C CNN
-F 2 "78XXL" H 10150 1500 20  0001 C CNN
+F 2 "Common:VREG_TO-220-3" H 10150 1500 20  0001 C CNN
 F 3 "" H 10150 1300 60  0001 C CNN
 F 4 "" H 10150 1481 60  0000 C CNN "Field4"
@@
 	9300 3500 9850 3500
 $Comp
-L power:GND #PWR?
+L power:GND #PWR0106
 U 1 1 60E98717
 P 6950 3200
-F 0 "#PWR?" H 6950 2950 50  0001 C CNN
+F 0 "#PWR0106" H 6950 2950 50  0001 C CNN
 F 1 "GND" H 6955 3027 50  0000 C CNN
 F 2 "" H 6950 3200 50  0001 C CNN
@@
 VALVE_SENSE
 $Comp
-L power:GND #PWR?
+L power:GND #PWR0107
 U 1 1 60FAB64F
 P 5450 7350
-F 0 "#PWR?" H 5450 7100 50  0001 C CNN
+F 0 "#PWR0107" H 5450 7100 50  0001 C CNN
 F 1 "GND" H 5455 7177 50  0000 C CNN
 F 2 "" H 5450 7350 50  0001 C CNN
@@
 	2050 3400 2650 3400
 $Comp
-L power:+12V #PWR?
+L power:+12V #PWR0108
 U 1 1 60E651F6
 P 10600 1150
-F 0 "#PWR?" H 10600 1000 50  0001 C CNN
+F 0 "#PWR0108" H 10600 1000 50  0001 C CNN
 F 1 "+12V" H 10615 1323 50  0000 C CNN
 F 2 "" H 10600 1150 50  0001 C CNN
@@
 	10600 1150 10600 1300
 $Comp
-L Connector_Generic:Conn_01x04 J?
+L Connector_Generic:Conn_01x04 J2
 U 1 1 60FA57D6
 P 5750 7050
-F 0 "J?" H 5830 7042 50  0000 L CNN
+F 0 "J2" H 5830 7042 50  0000 L CNN
 F 1 "Distance Sensor" H 5830 6951 50  0000 L CNN
 F 2 "" H 5750 7050 50  0001 C CNN
@@
 	9850 3500 10200 3500
 $Comp
-L SparkFun-PowerSymbols:3.3V #SUPPLY?
+L Tank_Sys-rescue:3.3V-SparkFun-PowerSymbols #SUPPLY0101
 U 1 1 60E95E58
 P 10200 3500
-F 0 "#SUPPLY?" H 10250 3500 45  0001 L BNN
+F 0 "#SUPPLY0101" H 10250 3500 45  0001 L BNN
 F 1 "3.3V" H 10200 3670 45  0000 C CNN
 F 2 "" H 10200 3681 60  0000 C CNN
@@
 $EndComp
 $Comp
-L SparkFun-PowerSymbols:3.3V #SUPPLY?
+L Tank_Sys-rescue:3.3V-SparkFun-PowerSymbols #SUPPLY0102
 U 1 1 60E6D9ED
 P 9650 1300
-F 0 "#SUPPLY?" H 9700 1300 45  0001 L BNN
+F 0 "#SUPPLY0102" H 9700 1300 45  0001 L BNN
 F 1 "3.3V" H 9650 1470 45  0000 C CNN
 F 2 "" H 9650 1481 60  0000 C CNN
@@
 	9850 1300 9650 1300
 $Comp
-L SparkFun-PowerSymbols:3.3V #SUPPLY?
+L Tank_Sys-rescue:3.3V-SparkFun-PowerSymbols #SUPPLY0103
 U 1 1 60E6F685
 P 5300 6850
-F 0 "#SUPPLY?" H 5350 6850 45  0001 L BNN
+F 0 "#SUPPLY0103" H 5350 6850 45  0001 L BNN
 F 1 "3.3V" H 5300 7020 45  0000 C CNN
 F 2 "" H 5300 7031 60  0000 C CNN
