File: KiCad/Common/Solenoid_Valve_Controller.sch (KiCad schematic (older format))
At the start: 9 parts

Commit message: Home update
Parts:
- SW2: renamed from SW?; footprint (none) -> Common:Switch_RA1153
- gave numbers to parts that had none: 8
Changed lines of the file:
@@
 $Descr A4 11693 8268
 encoding utf-8
-Sheet 3 19
+Sheet 3 3
 Title ""
 Date ""
@@
 P 5250 4400
 AR Path="/60FEC580" Ref="Q?"  Part="1"
-AR Path="/60FE860F/60FEC580" Ref="Q?"  Part="1"
+AR Path="/60FE860F/60FEC580" Ref="Q2"  Part="1"
 AR Path="/60E68C49/60FEC580" Ref="Q?"  Part="1"
 AR Path="/60E68E60/60FEC580" Ref="Q?"  Part="1"
@@
 AR Path="/60E699AB/60FEC580" Ref="Q?"  Part="1"
 AR Path="/60E699EC/60FEC580" Ref="Q?"  Part="1"
-F 0 "Q?" H 5454 4446 50  0000 L CNN
+F 0 "Q2" H 5454 4446 50  0000 L CNN
 F 1 "BS170" H 5454 4355 50  0000 L CNN
 F 2 "Package_TO_SOT_THT:TO-92_Inline" H 5450 4325 50  0001 L CIN
@@
 P 4850 3250
 AR Path="/60FEC586" Ref="M?"  Part="1"
-AR Path="/60FE860F/60FEC586" Ref="M?"  Part="1"
+AR Path="/60FE860F/60FEC586" Ref="M2"  Part="1"
 AR Path="/60E68C49/60FEC586" Ref="M?"  Part="1"
 AR Path="/60E68E60/60FEC586" Ref="M?"  Part="1"
@@
 AR Path="/60E699AB/60FEC586" Ref="M?"  Part="1"
 AR Path="/60E699EC/60FEC586" Ref="M?"  Part="1"
-F 0 "M?" H 5008 3246 50  0000 L CNN
+F 0 "M2" H 5008 3246 50  0000 L CNN
 F 1 "12V Solenoid Valve" H 5008 3155 50  0000 L CNN
 F 2 "" H 4850 3160 50  0001 C CNN
@@
 P 4500 3200
 AR Path="/60FEC5A2" Ref="D?"  Part="1"
-AR Path="/60FE860F/60FEC5A2" Ref="D?"  Part="1"
+AR Path="/60FE860F/60FEC5A2" Ref="D6"  Part="1"
 AR Path="/60E68C49/60FEC5A2" Ref="D?"  Part="1"
 AR Path="/60E68E60/60FEC5A2" Ref="D?"  Part="1"
@@
 AR Path="/60E699AB/60FEC5A2" Ref="D?"  Part="1"
 AR Path="/60E699EC/60FEC5A2" Ref="D?"  Part="1"
-F 0 "D?" V 4454 3280 50  0000 L CNN
+F 0 "D6" V 4454 3280 50  0000 L CNN
 F 1 "D" V 4545 3280 50  0000 L CNN
 F 2 "" H 4500 3200 50  0001 C CNN
@@
 P 4850 3900
 AR Path="/60FEC5B3" Ref="SW?"  Part="1"
-AR Path="/60FE860F/60FEC5B3" Ref="SW?"  Part="1"
+AR Path="/60FE860F/60FEC5B3" Ref="SW2"  Part="1"
 AR Path="/60E68C49/60FEC5B3" Ref="SW?"  Part="1"
 AR Path="/60E68E60/60FEC5B3" Ref="SW?"  Part="1"
@@
 AR Path="/60E699AB/60FEC5B3" Ref="SW?"  Part="1"
 AR Path="/60E699EC/60FEC5B3" Ref="SW?"  Part="1"
-F 0 "SW?" V 4896 4027 50  0000 L CNN
+F 0 "SW2" V 4896 4027 50  0000 L CNN
 F 1 "SW_SPDT" V 4805 3937 50  0000 L CNN
-F 2 "" H 4850 3900 50  0001 C CNN
+F 2 "Common:Switch_RA1153" H 4850 3900 50  0001 C CNN
 F 3 "~" H 4850 3900 50  0001 C CNN
 	1    4850 3900
@@
 AR Path="/60E699AB/610140FD" Ref="#PWR?"  Part="1"
 AR Path="/60E699EC/610140FD" Ref="#PWR?"  Part="1"
-AR Path="/60FE860F/610140FD" Ref="#PWR?"  Part="1"
-F 0 "#PWR?" H 4700 2750 50  0001 C CNN
+AR Path="/60FE860F/610140FD" Ref="#PWR0116"  Part="1"
+F 0 "#PWR0116" H 4700 2750 50  0001 C CNN
 F 1 "+12V" H 4715 3073 50  0000 C CNN
 F 2 "" H 4700 2900 50  0001 C CNN
@@
 AR Path="/60E699AB/6101484B" Ref="#PWR?"  Part="1"
 AR Path="/60E699EC/6101484B" Ref="#PWR?"  Part="1"
-AR Path="/60FE860F/6101484B" Ref="#PWR?"  Part="1"
-F 0 "#PWR?" H 4950 4400 50  0001 C CNN
+AR Path="/60FE860F/6101484B" Ref="#PWR0117"  Part="1"
+F 0 "#PWR0117" H 4950 4400 50  0001 C CNN
 F 1 "GND" H 4955 4477 50  0000 C CNN
 F 2 "" H 4950 4650 50  0001 C CNN
@@
 	4700 3000 4850 3000
 $Comp
-L Device:R R?
+L Device:R R4
 U 1 1 60EB80F6
 P 5500 4550
-F 0 "R?" H 5570 4596 50  0000 L CNN
+F 0 "R4" H 5570 4596 50  0000 L CNN
 F 1 "R" H 5570 4505 50  0000 L CNN
 F 2 "" V 5430 4550 50  0001 C CNN
@@
 	5500 4400 5600 4400
 $Comp
-L Device:LED D?
+L Device:LED D8
 U 1 1 60EB8B34
 P 5500 4900
-F 0 "D?" V 5539 4782 50  0000 R CNN
+F 0 "D8" V 5539 4782 50  0000 R CNN
 F 1 "LED" V 5448 4782 50  0000 R CNN
 F 2 "" H 5500 4900 50  0001 C CNN
@@
 AR Path="/60E699AB/60EBA2C3" Ref="#PWR?"  Part="1"
 AR Path="/60E699EC/60EBA2C3" Ref="#PWR?"  Part="1"
-AR Path="/60FE860F/60EBA2C3" Ref="#PWR?"  Part="1"
-F 0 "#PWR?" H 5500 4850 50  0001 C CNN
+AR Path="/60FE860F/60EBA2C3" Ref="#PWR0118"  Part="1"
+F 0 "#PWR0118" H 5500 4850 50  0001 C CNN
 F 1 "GND" H 5505 4927 50  0000 C CNN
 F 2 "" H 5500 5100 50  0001 C CNN
@@
 P 5100 3650
 AR Path="/60FEC599" Ref="D?"  Part="1"
-AR Path="/60FE860F/60FEC599" Ref="D?"  Part="1"
+AR Path="/60FE860F/60FEC599" Ref="D7"  Part="1"
 AR Path="/60E68C49/60FEC599" Ref="D?"  Part="1"
 AR Path="/60E68E60/60FEC599" Ref="D?"  Part="1"
@@
 AR Path="/60E699AB/60FEC599" Ref="D?"  Part="1"
 AR Path="/60E699EC/60FEC599" Ref="D?"  Part="1"
-F 0 "D?" V 5054 3730 50  0000 L CNN
+F 0 "D7" V 5054 3730 50  0000 L CNN
 F 1 "D" V 5145 3730 50  0000 L CNN
 F 2 "" H 5100 3650 50  0001 C CNN
@@
 VALVE_SENSE
 $Comp
-L Device:R R?
+L Device:R R3
 U 1 1 60ECB7E2
 P 4200 3150
-F 0 "R?" H 4270 3196 50  0000 L CNN
+F 0 "R3" H 4270 3196 50  0000 L CNN
 F 1 "R" H 4270 3105 50  0000 L CNN
 F 2 "" V 4130 3150 50  0001 C CNN
@@
 $EndComp
 $Comp
-L Device:LED D?
+L Device:LED D5
 U 1 1 60ECB7E8
 P 4200 3500
-F 0 "D?" V 4239 3382 50  0000 R CNN
+F 0 "D5" V 4239 3382 50  0000 R CNN
 F 1 "LED" V 4148 3382 50  0000 R CNN
 F 2 "" H 4200 3500 50  0001 C CNN

Commit message: Working Serial/MQTT connections
Changed lines of the file:
@@
 $Descr A4 11693 8268
 encoding utf-8
-Sheet 3 3
+Sheet 2 19
 Title ""
 Date ""
@@
 AR Path="/60E699AB/60FEC580" Ref="Q?"  Part="1"
 AR Path="/60E699EC/60FEC580" Ref="Q?"  Part="1"
-F 0 "Q2" H 5454 4446 50  0000 L CNN
+F 0 "Q?" H 5454 4446 50  0000 L CNN
 F 1 "BS170" H 5454 4355 50  0000 L CNN
 F 2 "Package_TO_SOT_THT:TO-92_Inline" H 5450 4325 50  0001 L CIN
@@
 AR Path="/60E699AB/60FEC586" Ref="M?"  Part="1"
 AR Path="/60E699EC/60FEC586" Ref="M?"  Part="1"
-F 0 "M2" H 5008 3246 50  0000 L CNN
+F 0 "M?" H 5008 3246 50  0000 L CNN
 F 1 "12V Solenoid Valve" H 5008 3155 50  0000 L CNN
 F 2 "" H 4850 3160 50  0001 C CNN
@@
 AR Path="/60E699AB/60FEC5A2" Ref="D?"  Part="1"
 AR Path="/60E699EC/60FEC5A2" Ref="D?"  Part="1"
-F 0 "D6" V 4454 3280 50  0000 L CNN
+F 0 "D?" V 4454 3280 50  0000 L CNN
 F 1 "D" V 4545 3280 50  0000 L CNN
 F 2 "" H 4500 3200 50  0001 C CNN
@@
 AR Path="/60E699AB/60FEC5B3" Ref="SW?"  Part="1"
 AR Path="/60E699EC/60FEC5B3" Ref="SW?"  Part="1"
-F 0 "SW2" V 4896 4027 50  0000 L CNN
+F 0 "SW?" V 4896 4027 50  0000 L CNN
 F 1 "SW_SPDT" V 4805 3937 50  0000 L CNN
 F 2 "Common:Switch_RA1153" H 4850 3900 50  0001 C CNN
@@
 AR Path="/60E699EC/610140FD" Ref="#PWR?"  Part="1"
 AR Path="/60FE860F/610140FD" Ref="#PWR0116"  Part="1"
-F 0 "#PWR0116" H 4700 2750 50  0001 C CNN
+F 0 "#PWR?" H 4700 2750 50  0001 C CNN
 F 1 "+12V" H 4715 3073 50  0000 C CNN
 F 2 "" H 4700 2900 50  0001 C CNN
@@
 AR Path="/60E699EC/6101484B" Ref="#PWR?"  Part="1"
 AR Path="/60FE860F/6101484B" Ref="#PWR0117"  Part="1"
-F 0 "#PWR0117" H 4950 4400 50  0001 C CNN
+F 0 "#PWR?" H 4950 4400 50  0001 C CNN
 F 1 "GND" H 4955 4477 50  0000 C CNN
 F 2 "" H 4950 4650 50  0001 C CNN
@@
 AR Path="/60E699EC/60EBA2C3" Ref="#PWR?"  Part="1"
 AR Path="/60FE860F/60EBA2C3" Ref="#PWR0118"  Part="1"
-F 0 "#PWR0118" H 5500 4850 50  0001 C CNN
+F 0 "#PWR?" H 5500 4850 50  0001 C CNN
 F 1 "GND" H 5505 4927 50  0000 C CNN
 F 2 "" H 5500 5100 50  0001 C CNN
@@
 AR Path="/60E699AB/60FEC599" Ref="D?"  Part="1"
 AR Path="/60E699EC/60FEC599" Ref="D?"  Part="1"
-F 0 "D7" V 5054 3730 50  0000 L CNN
+F 0 "D?" V 5054 3730 50  0000 L CNN
 F 1 "D" V 5145 3730 50  0000 L CNN
 F 2 "" H 5100 3650 50  0001 C CNN
