File: KiCad/Garden_Sys/Garden_Sys.sch (KiCad schematic (older format))
At the start: 5 parts

Commit message: Working Serial/MQTT connections
Parts:
- U?: symbol Arduino:Arduino_Pro_Mini -> Garden_Sys-rescue:Arduino_Pro_Mini-Arduino
- U?: symbol SparkFun-IC-Power:V_REG_LD1117VXX -> Garden_Sys-rescue:V_REG_LD1117VXX-SparkFun-IC-Power
- U?: symbol ESP8266:ESP-01v090 -> Garden_Sys-rescue:ESP-01v090-ESP8266
Changed lines of the file:
@@
 $EndDescr
 $Comp
-L Arduino:Arduino_Pro_Mini U?
+L Garden_Sys-rescue:Arduino_Pro_Mini-Arduino U?
 U 1 1 60E638E0
 P 2800 2500
@@
 $EndComp
 $Comp
-L SparkFun-IC-Power:V_REG_LD1117VXX U?
+L Garden_Sys-rescue:V_REG_LD1117VXX-SparkFun-IC-Power U?
 U 1 1 60E66743
 P 4300 1100
@@
 $EndComp
 $Comp
-L ESP8266:ESP-01v090 U?
+L Garden_Sys-rescue:ESP-01v090-ESP8266 U?
 U 1 1 60E67408
 P 5150 2350
