File: KiCad/Garden_Board/Garden_Board/Garden_Board.sch (KiCad schematic (older format))
At the start: 60 parts, among them J1 Barrel_Jack, J10 A1, J11 A2, J12 A3, J13 A4, J14 A5, J15 A6, J16 A7, J17 12V SWITCH P0 (Relay), J18 P0 RELAY BYPASS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

Commit message: Update Board V2 Darlington pair transistors for more current at ports, switching power supply for efficiency
Parts:
- removed J10: A1, Connector_PinHeader_2.54mm:PinHeader_1x03_P2.54mm_Vertical, symbol Connector_Generic:Conn_01x03
- removed J9: A0, Connector_PinHeader_2.54mm:PinHeader_1x03_P2.54mm_Vertical, symbol Connector_Generic:Conn_01x03
- removed U1: LD1117AV33, Package_TO_SOT_THT:TO-220-3_Vertical, symbol Regulator_Linear:LD1117S33TR_SOT223
- added C1: 100uF, Capacitor_THT:CP_Radial_D5.0mm_P2.00mm, symbol Device:CP1
- added C2: 1000uF, Capacitor_THT:CP_Radial_D10.0mm_P5.00mm, symbol Device:CP1
- added D21: MBR360, Diode_THT:D_DO-27_P12.70mm_Horizontal, symbol Device:D_Schottky
- added H1, H2, H3, H4: MountingHole, MountingHole:MountingHole_3.2mm_M3, symbol Mechanical:MountingHole
- added J6: ESP_TX_SEL, Connector_PinHeader_2.54mm:PinHeader_1x03_P2.54mm_Vertical, symbol Connector_Generic:Conn_01x03
- added J9: HC-SR04, Connector_PinHeader_2.54mm:PinHeader_1x04_P2.54mm_Vertical, symbol Connector_Generic:Conn_01x04
- added L1: 100uH, Inductor_THT:L_Radial_D9.5mm_P5.00mm_Fastron_07HVP, symbol Device:L
- added U1: LM2576HVS-3.3, Package_TO_SOT_THT:TO-220-5_Horizontal_TabDown, symbol Regulator_Switching:LM2576HVS-3.3
- D10, D11, D14, D15, D18, D19, D2, D3, D6, D7: footprint Diode_THT:D_DO-15_P10.16mm_Horizontal -> Diode_THT:D_DO-35_SOD27_P7.62mm_Horizontal
- J17: value 12V SWITCH P0 (Relay) -> P0
- J2: value 12V SWITCH P1 -> P1
- J4: value 12V SWITCH P2 -> P2
- J5: value ESP Serial -> ESP_RX_SEL
- J7: value 12V SWITCH P3 -> P3
- J8: value 12V SWITCH P4 -> P4
- Q1, Q2, Q4, Q5: value BS170-D75Z -> TIP12X; footprint Package_TO_SOT_THT:TO-92L_Inline -> Package_TO_SOT_THT:TO-220-3_Vertical; symbol Transistor_BJT:2N2219 -> Transistor_BJT:TIP122
- Q3: value NPN MOSFET -> TIP12X; footprint Package_TO_SOT_THT:TO-92L_Inline -> Package_TO_SOT_THT:TO-220-3_Vertical; symbol Transistor_BJT:2N2219 -> Transistor_BJT:TIP122
Connections:
- net +12V: now also C1.1, U1.1 (VIN); no longer U2.24 (RAW)
- net +3V3: now also U2.21 (VCC), C2.1, J9.1 (Pin_1), L1.2, U1.4 (FB)
- net CTRL0: now also Q5.1 (B); no longer Q5.2 (B)
- net CTRL1: now also Q1.1 (B); no longer Q1.2 (B)
- net CTRL2: now also Q2.1 (B); no longer Q2.2 (B)
- net CTRL3: now also Q3.1 (B); no longer Q3.2 (B)
- net CTRL4: now also Q4.1 (B); no longer Q4.2 (B)
- net ESP_RX: no longer U2.6 (~~D3)
- net ESP_TX: now also J6.2 (Pin_2); no longer J5.1 (Pin_1), U2.5 (D2)
- net GND: now also Q1.3 (E), Q2.3 (E), Q3.3 (E), Q4.3 (E), Q5.3 (E), C1.2, C2.2, D21.2 (A), J9.4 (Pin_4), U1.3 (GND), U1.5 (~ON~/OFF); no longer J5.3 (Pin_3), Q1.1 (E), Q2.1 (E), Q3.1 (E), Q4.1 (E), Q5.1 (E)
- net at J18.2 (Pin_2), K1.1: now also Q5.2 (C); no longer Q5.3 (C)
- net at SW1.3: now also Q1.2 (C); no longer Q1.3 (C)
- net at SW2.3: now also Q2.2 (C); no longer Q2.3 (C)
- net at SW3.3: now also Q3.2 (C); no longer Q3.3 (C)
- net at U2.1 (D1/TX): now also J6.1 (Pin_1)
- net at U2.2 (D0/RX): now also J5.1 (Pin_1)
- net at SW4.3: now also Q4.2 (C); no longer Q4.3 (C)
- net A0 renamed TRIG
- net TRIG: now also J9.2 (Pin_2)
- net A1 renamed ECHO
- net ECHO: now also J9.3 (Pin_3)
- new net: J6.3 (Pin_3), U2.5 (D2)
- new net: J5.3 (Pin_3), U2.6 (~~D3)
- new net: D21.1 (K), L1.1, U1.2 (OUT)
Other:
- moved on the sheet: J1, J3

Commit message: Mini Solenoid Unit
Parts:
- U2: symbol Arduino:Arduino_Pro_Mini -> Garden_Board-rescue:Arduino_Pro_Mini-Arduino
Changed lines of the file:
@@
 Connection ~ 9750 4650
 $Comp
-L Arduino:Arduino_Pro_Mini U2
+L Garden_Board-rescue:Arduino_Pro_Mini-Arduino U2
 U 1 1 622CD4AE
 P 4650 1800
